File: Main (2).kicad_sch (KiCad schematic)
At the start: 50 parts, among them J1-BATwGND1 Conn_01x02, J10 Conn_01x04, J11 Conn_01x02, J12 Conn_01x02, J13 Conn_01x02, J14 Conn_01x02, J15 Conn_01x02, J2-BATwMGND1 Conn_01x02, J3 Conn_01x04, J4 Conn_01x02, J5-servoPower1 Conn_01x02, J6 Conn_01x08_Socket, J7 Conn_01x08_Socket, J8 Conn_01x08_Socket, J9 Conn_01x08_Socket, Q1 PMOS, Q2 SS8050, U1 DEV-16771, U2 K230D, U4 AP63201WU, U6 AP63201WU

Commit message: Add files via upload
Parts:
- removed D4: 1N4148WT, Diode_SMD:D_SOD-523, symbol Diode:1N4148WT
- removed J15, J4, J5-servoPower1: Conn_01x02, Connector_TE-Connectivity:TE_440054-2_1x02_P2.00mm_Vertical, symbol Connector_Generic:Conn_01x02
Other:
- note removed: "led (?) then we can use 6.6v"
- note removed: "what on earth is J4"
