File: Main.kicad_pcb (KiCad board)
At the start: 2 copper layers, 83.5 x 82.8 mm, 32 parts, among them J1 Conn_01x02, J2 Conn_01x02, J3 Conn_01x06, J4 Conn_01x02, J5 Conn_01x02, J6 Conn_01x03, J7 Conn_01x04, U1 DEV-16771, U2 K230D, U3 SeeeduinoXIAO, U4 AP63201WU, U6 AP63201WU

Commit message: Add files via upload
Done, forgive the trace lengths or I die
Parts:
- added C11: 0.1uF, Capacitor_SMD:C_0603_1608Metric, B.Cu at (99.6, 97.1)
- added C12: 22uF, Capacitor_SMD:C_0603_1608Metric, B.Cu at (97.1, 97.1)
- added C13: 1uF, Capacitor_SMD:C_0603_1608Metric, B.Cu at (94.6, 97.1)
- added C14: 22uF, Capacitor_SMD:C_0603_1608Metric, F.Cu at (133.6, 93.0)
- added C15: 1uF, Capacitor_SMD:C_0603_1608Metric, F.Cu at (135.7, 93.0)
- added C16: 0.1uF, Capacitor_SMD:C_0603_1608Metric, F.Cu at (137.9, 93.0)
- added C17: 0.1uF, Capacitor_SMD:C_0603_1608Metric, F.Cu at (80.5, 108.8)
- added C18: 22uF, Capacitor_SMD:C_0603_1608Metric, F.Cu at (78.0, 108.8)
- added C19: 1uF, Capacitor_SMD:C_0603_1608Metric, F.Cu at (75.5, 108.8)
- added C20: 47uF, Capacitor_SMD:C_0603_1608Metric, F.Cu at (73.0, 108.8)
- added J8: Conn_01x03, Connector_TE-Connectivity:TE_826576-3_1x03_P3.96mm_Vertical, F.Cu at (141.5, 101.1)
- added J9: Conn_01x04, Connector_JST:JST_XH_B4B-XH-A_1x04_P2.50mm_Vertical, F.Cu at (128.6, 100.5)
- J3: value Conn_01x06 -> Conn_01x04; footprint Connector_TE-Connectivity:TE_826576-6_1x06_P3.96mm_Vertical -> Connector_JST:JST_XH_B4B-XH-A_1x04_P2.50mm_Vertical
- J7: footprint Connector_Stocko:Stocko_MKS_1654-6-0-404_1x4_P2.50mm_Vertical -> Connector_JST:JST_XH_B4B-XH-A_1x04_P2.50mm_Vertical
- U3: moved to B.Cu
- moved J3 76.7 mm to (73.0, 81.8), turned to 90 degrees
- moved J5 62.6 mm to (116.6, 132.4), turned to 180 degrees
- moved J2 61.7 mm to (109.1, 132.4), turned to 180 degrees
- moved J1 58.8 mm to (88.8, 131.7), turned to 180 degrees
- moved J4 58.2 mm to (77.6, 131.7), turned to 180 degrees
- moved U3 55.5 mm to (81.5, 104.7), turned to 90 degrees
- moved U1 48.3 mm to (108.7, 81.2), turned to 180 degrees
- moved D4 48.2 mm to (73.1, 124.0), turned to 0 degrees
- moved R8 46.2 mm to (102.3, 122.3), turned to 90 degrees
- moved D3 44.4 mm to (73.1, 121.6), turned to 0 degrees
- moved D2 40.8 mm to (73.1, 119.1), turned to 0 degrees
- moved U4 39.9 mm to (96.2, 122.5), turned to 180 degrees
- moved R6 39.8 mm to (102.4, 117.7), turned to 90 degrees
- moved C2 39.0 mm to (93.0, 123.3), turned to -90 degrees
- moved L1 38.7 mm to (89.8, 123.8), turned to 180 degrees
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Connections:
- J3 pad 1: /INT -> /SDA
- J3 pad 2: GND -> /SCL
- J3 pad 3: /SDA -> GND
- J3 pad 4: /SCL -> Net-(D1-K)
- U1 pad 2: /INT -> unconnected-(U1-OUT2-Pad2)
- U1 pad 20: unconnected-(U1-A6-Pad20) -> /AIN1
- U1 pad 21: unconnected-(U1-A7-Pad21) -> /AIN2
- U1 pad 22: unconnected-(U1-A8-Pad22) -> /PWMA
- U1 pad 24: /BIN2 -> unconnected-(U1-A10-Pad24)
- U1 pad 25: /BIN1 -> unconnected-(U1-A11-Pad25)
- U1 pad 26: /AIN2 -> unconnected-(U1-A12-Pad26)
- U1 pad 27: /AIN1 -> unconnected-(U1-A13-Pad27)
- U1 pad 3: unconnected-(U1-LRCLK2-Pad3) -> /BIN1_1
- U1 pad 3.3V_1: +3.3V -> Net-(U1-3.3V-Pad3.3V_1)
- U1 pad 3.3V_2: +3.3V -> Net-(U1-3.3V-Pad3.3V_1)
- U1 pad 3.3V_3: +3.3V -> Net-(U1-3.3V-Pad3.3V_1)
- U1 pad 30: unconnected-(U1-CRX3-Pad30) -> /AIN1_1
- U1 pad 31: unconnected-(U1-CTX3-Pad31) -> /AIN2_1
- U1 pad 33: unconnected-(U1-MCLK2-Pad33) -> /STBY_1
- U1 pad 36: unconnected-(U1-CS2-Pad36) -> /PWMB_1
- U1 pad 37: unconnected-(U1-CS3-Pad37) -> /PWMA_1
- U1 pad 39: /PWMA -> unconnected-(U1-A15-Pad39)
- U1 pad 4: unconnected-(U1-BCLK2-Pad4) -> /BIN2_1
- U1 pad 40: unconnected-(U1-A16-Pad40) -> /BIN1
- U1 pad 41: unconnected-(U1-A17-Pad41) -> /BIN2
- U1 pad VUSB: /VUSB -> unconnected-(U1-PadVUSB)
- U3 pad 13: unconnected-(U3-GND-Pad13) -> GND
Routing:
- net GND: track 211.4 -> 2.37 mm, vias 12 -> 5
- net /PWMB_1: track 0.00 -> 73.4 mm, vias 0 -> 1
- net /AIN1_1: track 0.00 -> 65.9 mm, vias 0 -> 4
- net /STBY_1: track 0.00 -> 63.2 mm, vias 0 -> 2
- net +3.3V: track 63.0 -> 0.00 mm
- net /AIN2_1: track 0.00 -> 62.2 mm, vias 0 -> 2
- net Net-(D1-K): track 74.1 -> 127.5 mm, vias 0 -> 1
- net /PWMA_1: track 0.00 -> 43.8 mm, vias 0 -> 1
- net /BIN2_1: track 0.00 -> 41.1 mm
- net +6.6V: track 103.2 -> 65.1 mm
- net /BIN1_1: track 0.00 -> 36.3 mm
- net /STBY: track 63.7 -> 27.4 mm, vias 3 -> 0
- net /INT: track 35.8 -> 0.00 mm
- net /SCL: track 27.5 -> 55.6 mm, vias 0 -> 6
- net /PWMB: track 26.5 -> 53.3 mm, vias 0 -> 2
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- added copper zone on B.Cu, net MGND
- removed copper zone on F.Cu, net +6.6V
Other:
- board size 83.5 x 82.8 mm -> 85.6 x 69.4 mm

Commit message: Add files via upload
Parts:
- removed C11: 0.1uF, Capacitor_SMD:C_0603_1608Metric
- removed C12: 22uF, Capacitor_SMD:C_0603_1608Metric
- removed C13: 1uF, Capacitor_SMD:C_0603_1608Metric
- removed U3: SeeeduinoXIAO, RF_Module:MCU_Seeed_ESP32C3
- added J10: Conn_01x04, Connector_JST:JST_XH_B4B-XH-A_1x04_P2.50mm_Vertical, F.Cu at (87.3, 59.1)
- moved C16 72.7 mm to (71.3, 63.9), turned to 180 degrees
- moved C15 71.6 mm to (71.3, 61.7), turned to 180 degrees
- moved C14 70.7 mm to (71.3, 59.6), turned to 180 degrees
- moved J8 49.3 mm to (116.5, 58.6), turned to 180 degrees
- moved J9 41.3 mm to (129.4, 59.2), turned to 180 degrees
- moved J3 36.5 mm to (101.6, 59.1), turned to 180 degrees
- moved J6 30.7 mm to (108.7, 87.1)
- moved J7 30.7 mm to (129.6, 87.7)
- moved U1 9.80 mm to (104.8, 72.2), turned to 0 degrees
- moved D2 3.13 mm to (73.2, 116.0)
- moved D1 2.13 mm to (73.2, 118.8)
- moved U2 2.05 mm to (96.7, 100.3)
- moved R8 1.41 mm to (103.7, 122.3)
- moved R6 1.41 mm to (103.8, 117.7)
Connections:
- U1 pad 20: /AIN1 -> /XIAO_TX
- U1 pad 21: /AIN2 -> /XIAO_RX
- U1 pad 22: /PWMA -> unconnected-(U1-A8-Pad22)
- U1 pad 23: /STBY -> unconnected-(U1-A9-Pad23)
- U1 pad 26: unconnected-(U1-A12-Pad26) -> /PWMB
- U1 pad 27: unconnected-(U1-A13-Pad27) -> /STBY
- U1 pad 28: /XIAO_TX -> /AIN1
- U1 pad 29: /XIAO_RX -> /AIN2
- U1 pad 3: /BIN1_1 -> unconnected-(U1-LRCLK2-Pad3)
- U1 pad 30: /AIN1_1 -> /PWMA
- U1 pad 31: /AIN2_1 -> /BIN1
- U1 pad 32: unconnected-(U1-OUT1B-Pad32) -> /BIN2
- U1 pad 33: /STBY_1 -> unconnected-(U1-MCLK2-Pad33)
- U1 pad 35: unconnected-(U1-TX8-Pad35) -> /PWMA_1
- U1 pad 36: /PWMB_1 -> /AIN2_1
- U1 pad 37: /PWMA_1 -> /AIN1_1
- U1 pad 38: /PWMB -> /STBY_1
- U1 pad 39: unconnected-(U1-A15-Pad39) -> /BIN1_1
- U1 pad 4: /BIN2_1 -> unconnected-(U1-BCLK2-Pad4)
- U1 pad 40: /BIN1 -> /BIN2_1
- U1 pad 41: /BIN2 -> /PWMB_1
Routing:
- net /PWMB_1: track 73.4 -> 8.11 mm, vias 1 -> 0
- net /AIN1_1: track 65.9 -> 5.70 mm, vias 4 -> 0
- net /STBY_1: track 63.2 -> 5.72 mm, vias 2 -> 0
- net /AIN2_1: track 62.2 -> 5.69 mm, vias 2 -> 0
- net Net-(U1-3.3V-Pad3.3V_1): track 0.00 -> 49.1 mm
- net /SCL: track 55.6 -> 8.08 mm, vias 6 -> 0
- net /PWMB: track 53.3 -> 8.07 mm, vias 2 -> 0
- net /BIN1: track 67.8 -> 25.7 mm, vias 3 -> 0
- net /XIAO_TX: track 48.7 -> 7.00 mm
- net /SDA: track 48.2 -> 8.04 mm, vias 2 -> 0
- net /PWMA_1: track 43.8 -> 5.67 mm, vias 1 -> 0
- net /PWMA: track 42.7 -> 8.10 mm, vias 1 -> 0
- net /BIN2_1: track 41.1 -> 7.52 mm
- net /BIN1_1: track 36.3 -> 6.93 mm
- net /AIN2: track 36.6 -> 8.11 mm
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Other:
- board size 85.6 x 69.4 mm -> 70 x 85.7 mm

Commit message: Add files via upload
I uploaded wrong versions I just saw
Parts:
- added J11: Conn_01x02, Connector_TE-Connectivity:TE_440054-2_1x02_P2.00mm_Vertical, F.Cu at (135.9, 77.9)
- added J12: Conn_01x02, Connector_TE-Connectivity:TE_440054-2_1x02_P2.00mm_Vertical, F.Cu at (103.5, 79.4)
- added J13: Conn_01x02, Connector_TE-Connectivity:TE_440054-2_1x02_P2.00mm_Vertical, F.Cu at (135.9, 85.1)
- added J14: Conn_01x02, Connector_TE-Connectivity:TE_440054-2_1x02_P2.00mm_Vertical, F.Cu at (103.5, 86.6)
- J6: value Conn_01x03 -> Conn_01x08_Socket; footprint Connector_TE-Connectivity:TE_826576-3_1x03_P3.96mm_Vertical -> Connector_PinHeader_2.54mm:PinHeader_1x08_P2.54mm_Vertical_SMD_Pin1Left
- J7: value Conn_01x04 -> Conn_01x08_Socket; footprint Connector_JST:JST_XH_B4B-XH-A_1x04_P2.50mm_Vertical -> Connector_PinHeader_2.54mm:PinHeader_1x08_P2.54mm_Vertical_SMD_Pin1Left
- J8: value Conn_01x03 -> Conn_01x08_Socket; footprint Connector_TE-Connectivity:TE_826576-3_1x03_P3.96mm_Vertical -> Connector_PinHeader_2.54mm:PinHeader_1x08_P2.54mm_Vertical_SMD_Pin1Left; moved to B.Cu
- J9: value Conn_01x04 -> Conn_01x08_Socket; footprint Connector_JST:JST_XH_B4B-XH-A_1x04_P2.50mm_Vertical -> Connector_PinHeader_2.54mm:PinHeader_1x08_P2.54mm_Vertical_SMD_Pin1Left; moved to B.Cu
- moved J8 32.4 mm to (120.2, 90.7), turned to 90 degrees
- moved J9 18.8 mm to (120.2, 75.5), turned to 90 degrees
- moved J7 15.4 mm to (120.2, 75.5), turned to 90 degrees
- moved J6 12.1 mm to (120.2, 90.7), turned to 90 degrees
- moved J10 10.2 mm to (87.5, 48.8)
- moved J3 10.2 mm to (101.8, 48.8)
- moved C14 10.2 mm to (71.5, 49.3)
- moved C15 10.2 mm to (71.5, 51.4)
- moved C16 10.2 mm to (71.5, 53.6)
- moved U1 10.2 mm to (105.0, 62.0)
Connections:
- C14 pad 1: Net-(D1-K) -> +5V
- C15 pad 1: Net-(D1-K) -> +5V
- C16 pad 1: Net-(D1-K) -> +5V
- D1 pad 1: Net-(D1-K) -> +5V
- J3 pad 4: Net-(D1-K) -> +5V
- J6 pad 1: /BIN1 -> MGND
- J6 pad 2: /BIN2 -> +5V
- J6 pad 3: /PWMB -> /AO1
- J8 pad 1: /BIN1_1 -> MGND
- J8 pad 2: /BIN2_1 -> +5V
- J8 pad 3: /PWMB_1 -> /AO1_1
- U1 pad 26: /PWMB -> /PWMA
- U1 pad 27: /STBY -> /AIN2
- U1 pad 28: /AIN1 -> /STBY
- U1 pad 29: /AIN2 -> /AIN1
- U1 pad 30: /PWMA -> /BIN2
- U1 pad 32: /BIN2 -> /PWMB
- U1 pad 5V: Net-(D1-K) -> +5V
- U1 pad VIN: Net-(D1-K) -> +5V
Routing:
- net +5V: track 0.00 -> 192.8 mm, vias 0 -> 5
- net MGND: track 0.00 -> 172.8 mm, vias 0 -> 4
- net Net-(D1-K): track 105.9 -> 0.00 mm
- net +6.6V: track 60.3 -> 113.0 mm, vias 2 -> 3
- net /AO1: track 0.00 -> 30.6 mm, vias 0 -> 2
- net /BO2: track 0.00 -> 29.7 mm, vias 0 -> 1
- net /BO1: track 0.00 -> 27.8 mm
- net /AO2: track 0.00 -> 22.2 mm, vias 0 -> 2
- net /BO2_1: track 0.00 -> 21.2 mm
- net /PWMA_1: track 5.67 -> 24.3 mm
- net /AIN1_1: track 5.70 -> 24.3 mm
- net /BIN1_1: track 6.93 -> 24.3 mm
- net /BIN2: track 24.3 -> 6.97 mm
- net /AO1_1: track 0.00 -> 17.2 mm
- net /PWMB_1: track 8.11 -> 24.3 mm
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Other:
- board size 70 x 85.7 mm -> 71.3 x 94.1 mm

Commit message: Add files via upload
Parts:
- added J15: Conn_01x02, Connector_TE-Connectivity:TE_440054-2_1x02_P2.00mm_Vertical, F.Cu at (126.1, 124.8)
- added Q1: PMOS, Package_TO_SOT_SMD:SOT-23, B.Cu at (85.3, 108.5)
- added Q2: SS8050, Package_TO_SOT_SMD:SOT-23, B.Cu at (85.2, 103.3)
- added R1: 1k, Resistor_SMD:R_0603_1608Metric, B.Cu at (85.2, 99.0)
- added R2: 1k, Resistor_SMD:R_0603_1608Metric, F.Cu at (84.2, 113.0)
- J12, J6, J7: moved to B.Cu
- moved J11 58.9 mm to (77.9, 88.0), turned to 90 degrees
- moved J14 33.6 mm to (135.9, 77.8), turned to -90 degrees
- moved J12 25.6 mm to (77.9, 78.6), turned to -90 degrees
- moved J6 22.4 mm to (97.8, 90.7)
- moved J7 22.4 mm to (97.8, 75.5)
- moved C8 0.89 mm to (81.4, 113.0)
- moved C4 0.73 mm to (86.8, 113.0)
Connections:
- D2 pad 2: +5.3V -> Net-(D2-A)
- U1 pad 10: unconnected-(U1-CS1-Pad10) -> /PWMA
- U1 pad 2: unconnected-(U1-OUT2-Pad2) -> /PWMB
- U1 pad 23: unconnected-(U1-A9-Pad23) -> /K230_ENABLE
- U1 pad 26: /PWMA -> unconnected-(U1-A12-Pad26)
- U1 pad 27: /AIN2 -> unconnected-(U1-A13-Pad27)
- U1 pad 28: /STBY -> unconnected-(U1-RX7-Pad28)
- U1 pad 29: /AIN1 -> unconnected-(U1-TX7-Pad29)
- U1 pad 3: unconnected-(U1-LRCLK2-Pad3) -> /BIN1
- U1 pad 30: /BIN2 -> unconnected-(U1-CRX3-Pad30)
- U1 pad 31: /BIN1 -> unconnected-(U1-CTX3-Pad31)
- U1 pad 32: /PWMB -> unconnected-(U1-OUT1B-Pad32)
- U1 pad 4: unconnected-(U1-BCLK2-Pad4) -> /BIN2
- U1 pad 5: unconnected-(U1-IN2-Pad5) -> /AIN1
- U1 pad 6: unconnected-(U1-OUT1D-Pad6) -> /STBY
- U1 pad 9: unconnected-(U1-OUT1C-Pad9) -> /AIN2
Routing:
- net /K230_ENABLE: track 0.00 -> 53.9 mm
- net +5.3V: track 0.00 -> 48.5 mm, vias 0 -> 2
- net MGND: track 172.8 -> 153.0 mm, vias 4 -> 5
- net Net-(D2-A): track 0.00 -> 17.6 mm, vias 0 -> 1
- net Net-(Q1-G): track 0.00 -> 11.0 mm, vias 0 -> 1
- net /BO1_1: track 13.9 -> 24.2 mm
- net /BO1: track 27.8 -> 20.4 mm
- net +6.6V: track 113.0 -> 119.9 mm, vias 3 -> 5
- net +5V: track 192.8 -> 186.4 mm, vias 5 -> 2
- net /AO2: track 22.2 -> 28.1 mm
- net /K230_RX: track 32.6 -> 38.5 mm
- net /AIN2: track 9.51 -> 5.52 mm
- net /PWMA: track 12.6 -> 8.83 mm
- net Net-(Q2-B): track 0.00 -> 3.43 mm
- net /AO1_1: track 17.2 -> 14.1 mm
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
Commit message: Add files via upload
Please help make smaller!
Parts:
- removed the J5 at (116.6, 132.4)
- added J10: Conn_01x03, Connector_JST:JST_XH_B3B-XH-A_1x03_P2.50mm_Vertical, B.Cu at (143.2, 52.8)
- added J11: Conn_01x06, Connector_JST:JST_XH_B6B-XH-AM_1x06_P2.50mm_Vertical, F.Cu at (116.2, 110.8)
- added J12: Conn_01x06, Connector_JST:JST_XH_B6B-XH-AM_1x06_P2.50mm_Vertical, F.Cu at (96.8, 110.9)
- added J13: Conn_01x06, Connector_JST:JST_XH_B6B-XH-AM_1x06_P2.50mm_Vertical, F.Cu at (96.8, 119.9)
- added J14: Conn_01x06, Connector_JST:JST_XH_B6B-XH-AM_1x06_P2.50mm_Vertical, F.Cu at (116.0, 119.9)
- added J16: Conn_01x06, Connector_JST:JST_XH_B6B-XH-AM_1x06_P2.50mm_Vertical, F.Cu at (115.8, 127.8)
- added J3: Conn_01x03, Connector_JST:JST_XH_B3B-XH-A_1x03_P2.50mm_Vertical, F.Cu at (112.7, 48.8)
- added J7: Conn_01x03, Connector_JST:JST_XH_B3B-XH-A_1x03_P2.50mm_Vertical, F.Cu at (135.5, 48.8)
- added J8: Conn_01x03, Connector_JST:JST_XH_B3B-XH-A_1x03_P2.50mm_Vertical, B.Cu at (143.2, 64.0)
- added J9: Conn_01x03, Connector_JST:JST_XH_B3B-XH-A_1x03_P2.50mm_Vertical, B.Cu at (143.2, 75.2)
- added S1: GF-126-0159, GF_126_0159:SW_GF-126-0159, F.Cu at (73.8, 125.3)
- added S2: GF-126-0159, GF_126_0159:SW_GF-126-0159, F.Cu at (140.1, 120.2)
- J15: value Conn_01x02 -> Conn_01x06; footprint Connector_TE-Connectivity:TE_440054-2_1x02_P2.00mm_Vertical -> Connector_JST:JST_XH_B6B-XH-AM_1x06_P2.50mm_Vertical
- J17: renamed from J11; moved to B.Cu
- J18: renamed from J12; moved to F.Cu
- J19: renamed from J13; moved to B.Cu
- J20: renamed from J14; moved to B.Cu
- J21: renamed from J8; footprint Connector_PinHeader_2.54mm:PinHeader_1x08_P2.54mm_Vertical_SMD_Pin1Left -> Connector_PinHeader_2.54mm:PinHeader_1x08_P2.54mm_Vertical; moved to F.Cu
- J22: renamed from J9; footprint Connector_PinHeader_2.54mm:PinHeader_1x08_P2.54mm_Vertical_SMD_Pin1Left -> Connector_PinHeader_2.54mm:PinHeader_1x08_P2.54mm_Vertical; moved to F.Cu
- J23: renamed from J6; footprint Connector_PinHeader_2.54mm:PinHeader_1x08_P2.54mm_Vertical_SMD_Pin1Left -> Connector_PinHeader_2.54mm:PinHeader_1x08_P2.54mm_Vertical; moved to F.Cu
- J24: renamed from J7; footprint Connector_PinHeader_2.54mm:PinHeader_1x08_P2.54mm_Vertical_SMD_Pin1Left -> Connector_PinHeader_2.54mm:PinHeader_1x08_P2.54mm_Vertical; moved to F.Cu
- J4: value Conn_01x02 -> Conn_01x03; footprint Connector_TE-Connectivity:TE_440054-2_1x02_P2.00mm_Vertical -> Connector_JST:JST_XH_B3B-XH-A_1x03_P2.50mm_Vertical
- L1, L2: footprint Inductor_SMD:L_0603_1608Metric -> Inductor_SMD:L_1210_3225Metric
- U2: moved to B.Cu
- moved J4 95.1 mm to (124.1, 48.8)
- moved J2 42.6 mm to (143.3, 107.0)
- moved J22 30.2 mm to (133.9, 102.4), turned to -90 degrees
- moved J24 30.1 mm to (111.5, 102.4), turned to -90 degrees
- moved J15 29.5 mm to (96.8, 128.0), turned to 0 degrees
- moved J18 23.0 mm to (87.8, 99.4), turned to 90 degrees
- moved J20 22.4 mm to (143.0, 99.0), turned to 90 degrees
- moved U2 20.9 mm to (97.6, 79.4)
- moved D4 14.3 mm to (68.5, 110.5)
- moved J21 14.1 mm to (133.9, 87.2), turned to -90 degrees
- moved J23 14.1 mm to (111.5, 87.2), turned to -90 degrees
- moved R6 13.3 mm to (92.1, 111.4)
- moved R8 13.3 mm to (92.0, 116.0)
- moved C7 12.7 mm to (80.7, 107.7)
- moved R5 12.6 mm to (80.6, 106.2)
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- renumbered J3 to J5, J10 to J6
Connections:
- J1 pad 1: +6.6V -> Net-(J1-Pin_1)
- J15 pad 1: +5.3V -> /X5
- J15 pad 2: GND -> /G5
- J2 pad 1: +6.6V -> Net-(J2-Pin_1)
- J4 pad 1: Net-(D4-K) -> GND
- J4 pad 2: GND -> /KRS2
- U1 pad 0: unconnected-(U1-RX1-Pad0) -> /G1
- U1 pad 1: unconnected-(U1-TX1-Pad1) -> /KRS1
- U1 pad 11: unconnected-(U1-MOSI-Pad11) -> /G6
- U1 pad 12: unconnected-(U1-MISO-Pad12) -> /X6
- U1 pad 13: unconnected-(U1-SCK-Pad13) -> /L1
- U1 pad 14: unconnected-(U1-A0-Pad14) -> /L2
- U1 pad 15: unconnected-(U1-A1-Pad15) -> /L3
- U1 pad 16: unconnected-(U1-A2-Pad16) -> /X3
- U1 pad 22: unconnected-(U1-A8-Pad22) -> /L4
- U1 pad 24: unconnected-(U1-A10-Pad24) -> /G4
- U1 pad 25: unconnected-(U1-A11-Pad25) -> /X4
- U1 pad 26: unconnected-(U1-A12-Pad26) -> /G5
- U1 pad 27: unconnected-(U1-A13-Pad27) -> /X5
- U1 pad 28: unconnected-(U1-RX7-Pad28) -> /X1
- U1 pad 29: unconnected-(U1-TX7-Pad29) -> /KRS2
- U1 pad 30: unconnected-(U1-CRX3-Pad30) -> /G2
- U1 pad 31: unconnected-(U1-CTX3-Pad31) -> /X2
- U1 pad 33: unconnected-(U1-MCLK2-Pad33) -> /G3
Routing:
- net +6.6V: track 119.9 -> 338.8 mm, vias 5 -> 1
- net /G4: track 0.00 -> 193.5 mm, vias 0 -> 6
- net /SDA: track 8.04 -> 196.5 mm
- net /SCL: track 8.08 -> 178.6 mm
- net /G1: track 0.00 -> 169.3 mm, vias 0 -> 2
- net /X6: track 0.00 -> 167.5 mm, vias 0 -> 4
- net /G6: track 0.00 -> 167.2 mm, vias 0 -> 6
- net /G5: track 0.00 -> 142.6 mm, vias 0 -> 5
- net /G2: track 0.00 -> 140.5 mm, vias 0 -> 3
- net /G3: track 0.00 -> 138.3 mm, vias 0 -> 2
- net MGND: track 153.0 -> 20.9 mm, vias 5 -> 7
- net Net-(D4-K): track 9.83 -> 109.6 mm, vias 0 -> 1
- net /X3: track 0.00 -> 86.3 mm, vias 0 -> 1
- net /X5: track 0.00 -> 84.7 mm, vias 0 -> 2
- net /PWMA: track 8.83 -> 78.0 mm
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- added copper zone on F.Cu, net MGND
Other:
- board size 71.3 x 94.1 mm -> 89.3 x 92.6 mm
