File: Main.kicad_sch (KiCad schematic)
At the start: 46 parts, among them J1 Conn_01x02, J2 Conn_01x02, J3 Conn_01x06, J4 Conn_01x02, J5 Conn_01x02, J6 Conn_01x03, J7 Conn_01x04, Q1 PMOS, Q2 NPN, Q3 PMOS, Q4 PMOS, Q5 PMOS, Q6 PMOS, Q7 PMOS, Q8 PMOS, Q9 PMOS, SW1 SW_Nidec_CAS-120A1, U1 DEV-16771, U2 K230D, U3 SeeeduinoXIAO, U4 AP63201WU, U6 AP63201WU

Commit message: Add files via upload
Main
Parts:
- removed Q1, Q3, Q4, Q5, Q6, Q7, Q8, Q9: PMOS, symbol Simulation_SPICE:PMOS
- removed Q2: NPN, symbol Simulation_SPICE:NPN
- removed R1, R2: 10k, symbol Device:R_US
- removed R3: 2k, symbol Device:R_US
- removed R4: 1k, symbol Device:R_US
- removed SW1: SW_Nidec_CAS-120A1, Button_Switch_SMD:Nidec_Copal_CAS-120A, symbol Switch:SW_Nidec_CAS-120A1
- J1, J2, J4, J5: footprint (none) -> Connector_TE-Connectivity:TE_440054-2_1x02_P2.00mm_Vertical
- J3: footprint (none) -> Connector_TE-Connectivity:TE_826576-6_1x06_P3.96mm_Vertical
- J6: footprint (none) -> Connector_TE-Connectivity:TE_826576-3_1x03_P3.96mm_Vertical
- J7: footprint (none) -> Connector_Stocko:Stocko_MKS_1654-6-0-404_1x4_P2.50mm_Vertical
- L1, L2: footprint (none) -> Inductor_SMD:L_0603_1608Metric
- R5, R6, R7, R8: footprint (none) -> Resistor_SMD:R_0603_1608Metric
- U1: footprint DEV-16771:MODULE_DEV-16771 -> Transformer_SMD:Teensy4.1
- U3: footprint (none) -> RF_Module:MCU_Seeed_ESP32C3
Connections:
- net +5V is gone; now on an unnamed net: U3.15 (5V)
- net K230_RX: now also U1.8 (TX2)
- net K230_TX: now also U1.7 (RX2)
- net XIAO_RX: now also U1.29 (TX7)
- net XIAO_TX: now also U1.28 (RX7)

Commit message: Add files via upload
Done, forgive the trace lengths or I die
Parts:
- removed J3: Conn_01x06, Connector_TE-Connectivity:TE_826576-6_1x06_P3.96mm_Vertical, symbol Connector_Generic:Conn_01x06
- added C11, C16, C17: 0.1uF, Capacitor_SMD:C_0603_1608Metric, symbol Device:C
- added C12, C14, C18: 22uF, Capacitor_SMD:C_0603_1608Metric, symbol Device:C
- added C13, C15, C19: 1uF, Capacitor_SMD:C_0603_1608Metric, symbol Device:C
- added C20: 47uF, Capacitor_SMD:C_0603_1608Metric, symbol Device:C
- added J3, J9: Conn_01x04, Connector_JST:JST_XH_B4B-XH-A_1x04_P2.50mm_Vertical, symbol Connector_Generic:Conn_01x04
- added J8: Conn_01x03, Connector_TE-Connectivity:TE_826576-3_1x03_P3.96mm_Vertical, symbol Connector_Generic:Conn_01x03
- J7: footprint Connector_Stocko:Stocko_MKS_1654-6-0-404_1x4_P2.50mm_Vertical -> Connector_JST:JST_XH_B4B-XH-A_1x04_P2.50mm_Vertical
Connections:
- net AIN1: now also U1.20 (A6); no longer U1.27 (A13)
- net AIN2: now also U1.21 (A7); no longer U1.26 (A12)
- net BIN1: now also U1.40 (A16); no longer U1.25 (A11)
- net BIN2: now also U1.41 (A17); no longer U1.24 (A10)
- net GND: now also U3.13 (GND), C11.2, C12.2, C13.2, C14.2, C15.2, C16.2, C17.2, C18.2, C19.2, C20.2, J3.3 (Pin_3)
- net PWMA: now also U1.22 (A8); no longer U1.39 (A15)
- net SCL: now also J3.2 (Pin_2)
- net SDA: now also J3.1 (Pin_1)
- net at D2.1 (K), U2.2 (5v), U2.4 (5v): now also C17.1, C18.1, C19.1, C20.1
- net at D3.1 (K), U3.14 (5V), U3.15 (5V): now also C11.1, C12.1, C13.1
- net at D1.1 (K), U1.5V, U1.VIN: now also C14.1, C15.1, C16.1, J3.4 (Pin_4)
- net BIN1_1: now reaches U1.3 (LRCLK2)
- net BIN1_1: now also J8.1 (Pin_1)
- net AIN1_1: now reaches U1.30 (CRX3)
- net AIN1_1: now also J9.3 (Pin_3)
- net AIN2_1: now reaches U1.31 (CTX3)
- net AIN2_1: now also J9.2 (Pin_2)
- net STBY_1: now reaches U1.33 (MCLK2)
- net STBY_1: now also J9.4 (Pin_4)
- net PWMB_1: now reaches U1.36 (CS2)
- net PWMB_1: now also J8.3 (Pin_3)
- net PWMA_1: now reaches U1.37 (CS3)
- net PWMA_1: now also J9.1 (Pin_1)
- net BIN2_1: now reaches U1.4 (BCLK2)
- net BIN2_1: now also J8.2 (Pin_2)
- net +3.3V: no longer names the net of U1.3.3V_1 (3.3V), U1.3.3V_2 (3.3V), U1.3.3V_3 (3.3V)
- net INT: no longer names the net of U1.2 (OUT2)
- net VUSB: no longer names the net of U1.VUSB
Other:
- moved on the sheet: D2, D3, U2

Commit message: Add files via upload
Parts:
- removed C11: 0.1uF, Capacitor_SMD:C_0603_1608Metric, symbol Device:C
- removed C12: 22uF, Capacitor_SMD:C_0603_1608Metric, symbol Device:C
- removed C13: 1uF, Capacitor_SMD:C_0603_1608Metric, symbol Device:C
- removed U3: SeeeduinoXIAO, RF_Module:MCU_Seeed_ESP32C3, symbol Seeeduino XIAO:SeeeduinoXIAO
- added J10: Conn_01x04, Connector_JST:JST_XH_B4B-XH-A_1x04_P2.50mm_Vertical, symbol Connector_Generic:Conn_01x04
Connections:
- net AIN1: now also U1.28 (RX7); no longer U1.20 (A6)
- net AIN1_1: now also U1.37 (CS3); no longer U1.30 (CRX3)
- net AIN2: now also U1.29 (TX7); no longer U1.21 (A7)
- net AIN2_1: now also U1.36 (CS2); no longer U1.31 (CTX3)
- net BIN1: now also U1.31 (CTX3); no longer U1.40 (A16)
- net BIN1_1: now also U1.39 (A15); no longer U1.3 (LRCLK2)
- net BIN2: now also U1.32 (OUT1B); no longer U1.41 (A17)
- net BIN2_1: now also U1.40 (A16); no longer U1.4 (BCLK2)
- net GND: now also J10.3 (Pin_3)
- net PWMA: now also U1.30 (CRX3); no longer U1.22 (A8)
- net PWMA_1: now also U1.35 (TX8); no longer U1.37 (CS3)
- net PWMB: now also U1.26 (A12); no longer U1.38 (A14)
- net PWMB_1: now also U1.41 (A17); no longer U1.36 (CS2)
- net STBY: now also U1.27 (A13); no longer U1.23 (A9)
- net STBY_1: now also U1.38 (A14); no longer U1.33 (MCLK2)
- net XIAO_RX: now also U1.21 (A7), J10.2 (Pin_2); no longer U1.29 (TX7)
- net XIAO_TX: now also U1.20 (A6), J10.1 (Pin_1); no longer U1.28 (RX7)
- net at D3.1 (K): now also J10.4 (Pin_4)
Other:
- moved on the sheet: D3

Commit message: Add files via upload
I uploaded wrong versions I just saw
Parts:
- removed J2: Conn_01x02, Connector_TE-Connectivity:TE_440054-2_1x02_P2.00mm_Vertical, symbol Connector_Generic:Conn_01x02
- removed J6, J8: Conn_01x03, Connector_TE-Connectivity:TE_826576-3_1x03_P3.96mm_Vertical, symbol Connector_Generic:Conn_01x03
- removed J7, J9: Conn_01x04, Connector_JST:JST_XH_B4B-XH-A_1x04_P2.50mm_Vertical, symbol Connector_Generic:Conn_01x04
- added J11, J12, J13, J14: Conn_01x02, Connector_TE-Connectivity:TE_440054-2_1x02_P2.00mm_Vertical, symbol Connector_Generic:Conn_01x02
- added J6, J7, J8, J9: Conn_01x08_Socket, Connector_PinHeader_2.54mm:PinHeader_1x08_P2.54mm_Vertical_SMD_Pin1Left, symbol Connector:Conn_01x08_Socket
Connections:
- net +6.6V: now also J6.7 (Pin_7), J8.7 (Pin_7)
- net AIN1: now also U1.29 (TX7), J7.3 (Pin_3); no longer U1.28 (RX7)
- net AIN1_1: now also J9.3 (Pin_3)
- net AIN2: now also U1.27 (A13), J7.2 (Pin_2); no longer U1.29 (TX7)
- net AIN2_1: now also J9.2 (Pin_2)
- net BIN1: now also J7.5 (Pin_5)
- net BIN1_1: now also J9.5 (Pin_5)
- net BIN2: now also U1.30 (CRX3), J7.6 (Pin_6); no longer U1.32 (OUT1B)
- net BIN2_1: now also J9.6 (Pin_6)
- net GND: now also J6.1 (Pin_1), J6.8 (Pin_8), J7.8 (Pin_8), J8.1 (Pin_1), J8.8 (Pin_8), J9.8 (Pin_8)
- net PWMA: now also U1.26 (A12), J7.1 (Pin_1); no longer U1.30 (CRX3)
- net PWMA_1: now also J9.1 (Pin_1)
- net PWMB: now also U1.32 (OUT1B), J7.7 (Pin_7); no longer U1.26 (A12)
- net PWMB_1: now also J9.7 (Pin_7)
- net STBY: now also U1.28 (RX7), J7.4 (Pin_4); no longer U1.27 (A13)
- net STBY_1: now also J9.4 (Pin_4)
- net +5V: now reaches C14.1, C15.1, C16.1, D1.1 (K), J3.4 (Pin_4), U1.5V, U1.VIN
- net +5V: now also J6.2 (Pin_2), J8.2 (Pin_2)
- new net AO1: J11.1 (Pin_1), J6.3 (Pin_3)
- new net AO1_1: J13.1 (Pin_1), J8.3 (Pin_3)
- new net AO2: J11.2 (Pin_2), J6.4 (Pin_4)
- new net AO2_1: J13.2 (Pin_2), J8.4 (Pin_4)
- new net BO1: J12.1 (Pin_1), J6.6 (Pin_6)
- new net BO1_1: J14.1 (Pin_1), J8.6 (Pin_6)
- new net BO2: J12.2 (Pin_2), J6.5 (Pin_5)
- new net BO2_1: J14.2 (Pin_2), J8.5 (Pin_5)

Commit message: Add files via upload
Parts:
- added J15, J2: Conn_01x02, Connector_TE-Connectivity:TE_440054-2_1x02_P2.00mm_Vertical, symbol Connector_Generic:Conn_01x02
- added Q1: PMOS, Package_TO_SOT_SMD:SOT-23, symbol Simulation_SPICE:PMOS
- added Q2: SS8050, Package_TO_SOT_SMD:SOT-23, symbol Transistor_BJT:SS8050
- added R1, R2: 1k, Resistor_SMD:R_0603_1608Metric, symbol Device:R_US
Connections:
- net +5.3V: now also J15.1 (Pin_1), Q1.1 (D), R2.1; no longer D2.2 (A)
- net +6.6V: now also J2.1 (Pin_1)
- net AIN1: now also U1.5 (IN2); no longer U1.29 (TX7)
- net AIN2: now also U1.9 (OUT1C); no longer U1.27 (A13)
- net AO1_1: now also J13.2 (Pin_2); no longer J13.1 (Pin_1)
- net AO2_1: now also J13.1 (Pin_1); no longer J13.2 (Pin_2)
- net BIN1: now also U1.3 (LRCLK2); no longer U1.31 (CTX3)
- net BIN2: now also U1.4 (BCLK2); no longer U1.30 (CRX3)
- net GND: now also J15.2 (Pin_2), Q2.2 (E); no longer J6.1 (Pin_1), J6.8 (Pin_8), J7.8 (Pin_8), J8.1 (Pin_1), J8.8 (Pin_8), J9.8 (Pin_8)
- net MGND: now also J6.1 (Pin_1), J6.8 (Pin_8), J7.8 (Pin_8), J8.1 (Pin_1), J8.8 (Pin_8), J9.8 (Pin_8), J2.2 (Pin_2)
- net PWMA: now also U1.10 (CS1); no longer U1.26 (A12)
- net PWMB: now also U1.2 (OUT2); no longer U1.32 (OUT1B)
- net STBY: now also U1.6 (OUT1D); no longer U1.28 (RX7)
- net K230_ENABLE: now reaches U1.23 (A9)
- net K230_ENABLE: now also R1.1
- new net: Q2.1 (B), R1.2
- new net: Q1.2 (G), Q2.3 (C), R2.2
- new net: D2.2 (A), Q1.3 (S)
Other:
- moved on the sheet: J5

Commit message: Add files via upload
Please help make smaller!
Parts:
- removed J15, J4, J5: Conn_01x02, Connector_TE-Connectivity:TE_440054-2_1x02_P2.00mm_Vertical, symbol Connector_Generic:Conn_01x02
- added J10, J3, J4, J7, J8, J9: Conn_01x03, Connector_JST:JST_XH_B3B-XH-A_1x03_P2.50mm_Vertical, symbol Connector_Generic:Conn_01x03
- added J11, J12, J13, J14, J15, J16: Conn_01x06, Connector_JST:JST_XH_B6B-XH-AM_1x06_P2.50mm_Vertical, symbol Connector_Generic:Conn_01x06
- added S1, S2: GF-126-0159, GF_126_0159:SW_GF-126-0159, symbol GF-126-0159:GF-126-0159
- J21: renamed from J8; footprint Connector_PinHeader_2.54mm:PinHeader_1x08_P2.54mm_Vertical_SMD_Pin1Left -> Connector_PinHeader_2.54mm:PinHeader_1x08_P2.54mm_Vertical
- J22: renamed from J9; footprint Connector_PinHeader_2.54mm:PinHeader_1x08_P2.54mm_Vertical_SMD_Pin1Left -> Connector_PinHeader_2.54mm:PinHeader_1x08_P2.54mm_Vertical
- J23: renamed from J6; footprint Connector_PinHeader_2.54mm:PinHeader_1x08_P2.54mm_Vertical_SMD_Pin1Left -> Connector_PinHeader_2.54mm:PinHeader_1x08_P2.54mm_Vertical
- J24: renamed from J7; footprint Connector_PinHeader_2.54mm:PinHeader_1x08_P2.54mm_Vertical_SMD_Pin1Left -> Connector_PinHeader_2.54mm:PinHeader_1x08_P2.54mm_Vertical
- L1, L2: footprint Inductor_SMD:L_0603_1608Metric -> Inductor_SMD:L_1210_3225Metric
- renumbered J11 to J17, J12 to J18, J13 to J19, J14 to J20, J3 to J5, J10 to J6
Connections:
- net +6.6V: now also J10.3 (Pin_3), J3.3 (Pin_3), J4.3 (Pin_3), J7.3 (Pin_3), J8.3 (Pin_3), J9.3 (Pin_3), S1.1, S1.4, S2.1, S2.4; no longer J1.1 (Pin_1), J2.1 (Pin_1)
- net GND: now also J10.1 (Pin_1), J11.5 (Pin_5), J12.5 (Pin_5), J13.5 (Pin_5), J14.5 (Pin_5), J15.5 (Pin_5), J16.5 (Pin_5), J3.1 (Pin_1), J4.1 (Pin_1), J7.1 (Pin_1), J8.1 (Pin_1), J9.1 (Pin_1)
- net SCL: now also J11.4 (Pin_4), J12.4 (Pin_4), J13.4 (Pin_4), J14.4 (Pin_4), J15.4 (Pin_4), J16.4 (Pin_4)
- net SDA: now also J11.3 (Pin_3), J12.3 (Pin_3), J13.3 (Pin_3), J14.3 (Pin_3), J15.3 (Pin_3), J16.3 (Pin_3)
- net at D4.1 (K): now also J11.6 (Pin_6), J12.6 (Pin_6), J13.6 (Pin_6), J14.6 (Pin_6), J15.6 (Pin_6), J16.6 (Pin_6)
- net G1: now reaches U1.0 (RX1)
- net G1: now also J11.2 (Pin_2)
- net KRS1: now reaches U1.1 (TX1)
- net KRS1: now also J3.2 (Pin_2)
- net G6: now reaches U1.11 (MOSI)
- net G6: now also J16.2 (Pin_2)
- net X6: now reaches U1.12 (MISO)
- net X6: now also J16.1 (Pin_1)
- net L1: now reaches U1.13 (SCK)
- net L1: now also J7.2 (Pin_2)
- net L2: now reaches U1.14 (A0)
- net L2: now also J8.2 (Pin_2)
- net L3: now reaches U1.15 (A1)
- net L3: now also J9.2 (Pin_2)
- net X3: now reaches U1.16 (A2)
- net X3: now also J13.1 (Pin_1)
- net L4: now reaches U1.22 (A8)
- net L4: now also J10.2 (Pin_2)
- net G4: now reaches U1.24 (A10)
- net G4: now also J14.2 (Pin_2)
- net X4: now reaches U1.25 (A11)
- net X4: now also J14.1 (Pin_1)
- net G5: now reaches U1.26 (A12)
- net G5: now also J15.2 (Pin_2)
- net X5: now reaches U1.27 (A13)
- net X5: now also J15.1 (Pin_1)
- net X1: now reaches U1.28 (RX7)
- net X1: now also J11.1 (Pin_1)
- net KRS2: now reaches U1.29 (TX7)
- net KRS2: now also J4.2 (Pin_2)
- net G2: now reaches U1.30 (CRX3)
- net G2: now also J12.2 (Pin_2)
- net X2: now reaches U1.31 (CTX3)
- net X2: now also J12.1 (Pin_1)
- net G3: now reaches U1.33 (MCLK2)
- net G3: now also J13.2 (Pin_2)
- new net: J1.1 (Pin_1), S1.2, S1.5
- new net: J2.1 (Pin_1), S2.2, S2.5
Other:
- note added: "MOTOR"
- note added: "Regulators"
- note added: "XIAO"
- company: (none) -> FATEN Robotics
- title: (none) -> Main PCB Schematic
- moved on the sheet: C1, C10, C14, C15, C16, C17, C18, C19, C2, C20, C3, C4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
