File: Electronics/powermanagmen/powermanagmen.kicad_sch (KiCad schematic)
At the start: 28 parts, among them J1 STS3032, J10 buzzer, J11 Line LED, J12 STS3032, J13 STS3032, J14 STS3032, J2 KRS3301, J3 HS45HB-0, J4 HS45HB-1, J5 IMU MPU6050, J6 touch, J7 touch, J8 conductive-0, J9 conductive-0, U1 74LS126, U2 K230D, U3 DEV-16771

Commit message: powermanagmen
Parts:
- added C17, C4: 0.1uF, Capacitor_SMD:C_0603_1608Metric, symbol Device:C
- added C18, C3: 1uF, Capacitor_SMD:C_0603_1608Metric, symbol Device:C
- added C19, C2: 22uF, Capacitor_SMD:C_0603_1608Metric, symbol Device:C
- added C20: 47uF, Capacitor_SMD:C_0603_1608Metric, symbol Device:C
- added D1, D2: 1N4148WT, Diode_SMD:D_SOD-523, symbol Diode:1N4148WT
- added J15: 3.3V, symbol Connector:Conn_01x02_Socket
- added J16, J17: 5.3V, symbol Connector:Conn_01x02_Socket
- added J18, J25, J26, J27, J28, J29: VL53L0X, symbol Connector:Conn_01x05_Socket
- added J31: XIAO-esp32, Connector_JST:JST_XH_B4B-XH-A_1x04_P2.50mm_Vertical, symbol Connector:Conn_01x04_Socket
- added Q1: PMOS, Package_TO_SOT_SMD:SOT-23, symbol Simulation_SPICE:PMOS
- added Q2: SS8050, Package_TO_SOT_SMD:SOT-23, symbol Transistor_BJT:SS8050
- added R13, R14: 1k, Resistor_SMD:R_0603_1608Metric, symbol Device:R_US
- J11: value Line LED -> LED-Output
- R4, R5, R6, R7: value 1k -> 330 to 1k
Connections:
- net Teensy 6? is gone; now on net Teensy any pin: R5.2
- net Teensy 7? is gone; now on net Teensy any pin: R6.2
- net +3.3V: now also R2.1, R3.1, J15.1 (Pin_1), J18.1 (Pin_1), J25.1 (Pin_1), J26.1 (Pin_1), J27.1 (Pin_1), J28.1 (Pin_1), J29.1 (Pin_1); no longer R2.2, R3.2
- net +5V: now also U3.5V, D1.1 (K)
- net +6.6V: now also J11.1 (Pin_1), J17.1 (Pin_1)
- net GND: now also J11.2 (Pin_2), C17.2, C18.2, C19.2, C2.1, C20.2, C3.1, C4.1, J15.2 (Pin_2), J16.2 (Pin_2), J17.2 (Pin_2), J18.2 (Pin_2), J25.2 (Pin_2), J26.2 (Pin_2), J27.2 (Pin_2), J28.2 (Pin_2), J29.2 (Pin_2), J31.4 (Pin_4), Q2.2 (E)
- net Teensy 8?: no longer R7.2
- net Teensy SCL-0: now also R3.2; no longer R3.1
- net Teensy SDA-0: now also R2.2; no longer R2.1
- net at U2.2 (5v): now also U2.4 (5v), C17.1, C18.1, C19.1, C20.1, D2.1 (K)
- net at U3.VIN: now also C2.2, C3.2, C4.2
- net Teensy 5? renamed Teensy any pin
- net Teensy any pin: now also R7.2
- new net: Q2.1 (B), R14.2
- new net: Q1.2 (G), Q2.3 (C), R13.2
- new net: D2.2 (A), Q1.3 (S)
- new net +5.3V: D1.2 (A), J16.1 (Pin_1), J31.3 (Pin_3), Q1.1 (D), R13.1
- new net Teensy KRS Enable: R14.1
- new net Teensy SCL-1: J18.4 (Pin_4), J25.4 (Pin_4), J26.4 (Pin_4), J27.4 (Pin_4), J28.4 (Pin_4), J29.4 (Pin_4)
- new net Teensy SDA-1: J18.3 (Pin_3), J25.3 (Pin_3), J26.3 (Pin_3), J27.3 (Pin_3), J28.3 (Pin_3), J29.3 (Pin_3)
- new net Teensy d?: J18.5 (Pin_5), J25.5 (Pin_5), J26.5 (Pin_5), J27.5 (Pin_5), J28.5 (Pin_5), J29.5 (Pin_5)
- new net XIAO_RX: J31.2 (Pin_2)
- new net XIAO_TX: J31.1 (Pin_1)
Other:
- note added: "connector footprint could be diff"
- note added: "voltage divider"
- note added: "xt60?"
- note removed: "voltage divider, urat k230 esp-xiao, vl53l0x start ground able to turn k230 off at non-evac area"
- moved on the sheet: J1, J10, J12, J13, J14, J2, J3, J4, J5, J6, J7, J8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

Commit message: powermanagmen merged all circuit
Parts:
- added C10, C13, C14: 100pF, Capacitor_SMD:C_0603_1608Metric, symbol Device:C
- added C10, C6, C9: 10uF, Capacitor_SMD:C_0603_1608Metric, symbol Device:C
- added C10, C11, C15, C16, C21, C9: 22uF, Capacitor_SMD:C_0603_1608Metric, symbol Device:C
- added C11, C12, C9: 100nF, Capacitor_SMD:C_0603_1608Metric, symbol Device:C
- added C12: 150pF, symbol Device:C_Small
- added C5, C7: 10uF, symbol Device:C_Small
- added C5, C8: 0.1uF, symbol Device:C_Small
- added C6, C7, C8: 22uF, symbol Device:C_Small
- added D?: 1N4148WT, Diode_SMD:D_SOD-523, symbol Diode:1N4148WT
- added J19, J20: Conn_01x02, Connector_Molex:Molex_KK-396_A-41791-0002_1x02_P3.96mm_Vertical, symbol Connector_Generic:Conn_01x02
- added J?: XIAO-esp32, Connector_JST:JST_XH_B4B-XH-A_1x04_P2.50mm_Vertical, symbol Connector:Conn_01x04_Socket
- added L1: 3.3uH, symbol Device:L
- added L2 (x2): 10uH, Inductor_SMD:L_1210_3225Metric, symbol Device:L
- added L3: 6.8uH, Inductor_SMD:L_1210_3225Metric, symbol Device:L
- added R11: 52.3k, symbol Device:R_US
- added R12: 196k, Resistor_SMD:R_0603_1608Metric, symbol Device:R_US
- added R15: 62k, Resistor_SMD:R_0603_1608Metric, symbol Device:R_US
- added R16, R18: 169k, Resistor_SMD:R_0603_1608Metric, symbol Device:R_US
- added R17, R19: 30k, Resistor_SMD:R_0603_1608Metric, symbol Device:R_US
- added R20: 90k, symbol Device:R_US
- added R21: 10k, symbol Device:R_US
- added S1, S2: GF-126-0159, GF_126_0159:SW_GF-126-0159, symbol GF-126-0159:GF-126-0159
- added U4, U6, U7: AP63201WU, Package_TO_SOT_SMD:TSOT-23-6, symbol Regulator_Switching:AP63201WU
- added U5: TPS56A37RPAR, Audio_Module:RPA0010A-MFG, symbol 2026-01-05_00-17-44:TPS56A37RPAR
Connections:
- net GND is gone; now on net AGND: C1.1, C17.2, C18.2, C19.2, C2.1, C20.2, C3.1, C4.1, J10.2 (Pin_2), J11.2 (Pin_2), J15.2 (Pin_2), J16.2 (Pin_2), J17.2 (Pin_2), J18.2 (Pin_2), J2.3 (Pin_3), J25.2 (Pin_2), J26.2 (Pin_2), J27.2 (Pin_2), J28.2 (Pin_2), J29.2 (Pin_2), J3.3 (Pin_3), J31.4 (Pin_4), J4.3 (Pin_3), J5.1 (Pin_1), J6.2 (Pin_2), J7.2 (Pin_2), J8.2 (Pin_2), J9.2 (Pin_2), Q2.2 (E), R1.1, R10.2, U1.7 (GND)
- net MGND is gone; now on net AGND: J1.3 (Pin_3), J12.3 (Pin_3), J13.3 (Pin_3), J14.3 (Pin_3)
- net +3.3V: now also C10.1, C11.1, C21.1, L3.2, R12.1
- net +5.3V: now also C10.1, C13.1, C14.1, C15.1, C16.1, C9.1, L2.2, L2.2, R16.1, R18.1
- net +5V: now also D?.1 (K)
- net +6V: now also C12.1, C6.1, C7.1, C8.1, L1.2, R20.1
- net AGND: now reaches U2.14 (GND)
- net AGND: now also U2.20 (GND), U2.25 (GND), U2.30 (GND), U2.34 (GND), U2.39 (GND), U2.6 (GND), U2.9 (GND), U3.GND1 (GND), U3.GND2 (GND), U3.GND3 (GND), U3.GND4 (GND), U3.GND5 (GND), C10.2, C10.2, C11.2, C15.2, C16.2, C21.2, C6.2, C6.2, C7.2, C8.2, C9.2, C9.2, J19.2 (Pin_2), J20.2 (Pin_2), J?.1 (Pin_1), R11.2, R15.2, R17.2, R19.2, R21.2, U4.4 (GND), U5.3 (AGND), U5.9 (PGND), U6.4 (GND), U7.4 (GND)
- new net: C11.2, L2.1, U6.6 (BST)
- new net: J20.1 (Pin_1), S1.2, S1.5
- new net: C14.2, R18.2, R19.1, U7.1 (FB)
- new net: C12.2, R20.2, R21.1, U5.2 (FB)
- new net: C12.1, U7.5 (SW)
- new net: C12.2, L2.1, U7.6 (BST)
- new net: C10.2, R12.2, R15.1, U4.1 (FB)
- new net: C9.2, L3.1, U4.6 (BST)
- new net: C13.2, R16.2, R17.1, U6.1 (FB)
- new net: C9.1, U4.5 (SW)
- new net: C11.1, U6.5 (SW)
- new net: C5.2, C7.2, C8.2
- new net: D?.2 (A), J?.2 (Pin_2)
- new net: R11.1, U5.10 (MODE)
- new net: C5.2, L1.1, U5.6 (SW)
- new net: C5.1, U5.7 (BOOT)
- new net: J19.1 (Pin_1), S2.2, S2.5
- new net +BATT: C10.1, C5.1, C6.1, C7.1, C8.1, C9.1, S1.1, S1.4, S2.1, S2.4, U4.2 (EN), U4.3 (IN), U5.1 (EN), U5.8 (VIN), U6.2 (EN), U6.3 (IN), U7.2 (EN), U7.3 (IN)
Other:
- note added: "Power Switches"
- note added: "Regulators"
- note added: "voltage divider assign ports. pwer works. pcb layout"
- note removed: "voltage divider"
- moved on the sheet: C17, C18, C19, C20, D2, Q1, Q2, R13, R14, U2

Commit message: kicad update
Parts:
- removed D1, D2, D?: 1N4148WT, Diode_SMD:D_SOD-523, symbol Diode:1N4148WT
- added D?: 1N4148WT, Diode_SMD:D_SOD-523, symbol Diode:1N4148WT
Connections:
- net +5.3V: no longer Q1.1 (D), R13.1
- net +5V: now also J?.2 (Pin_2), Q1.1 (D), R13.1; no longer J3.1 (Pin_1), J4.1 (Pin_1)
- net +6V: now also J3.1 (Pin_1), J4.1 (Pin_1)
- net at C17.1, C18.1, C19.1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: now also Q1.3 (S)
- net Teensy 8? renamed K230D pin?
- net XIAO_RX: no longer names the net of J31.2 (Pin_2)
- net XIAO_RX: now also D?.1 (K)
- net XIAO_TX renamed Teensy TX2?
- new net Teensy RX2?: D?.2 (A)
Other:
- moved on the sheet: C2, C3, C4, U3
